Commit message: allowing simulation env to run Kinetic and operators front end

File: cyton_gamma_300_description/cyton_gamma_300.urdf (robot description, URDF)
Before this commit: robot cyton_gamma_300, 12 links, 11 joints
Links:
- removed link gripper_finger1
- removed link gripper_finger2
- link base_link: mass None -> 100.0
- link elbow_pitch: mass None -> 10.0
- link elbow_roll: mass None -> 10.0
- link elbow_yaw: mass None -> 10.0
- link shoulder_pitch: mass None -> 20.0
- link shoulder_roll: mass None -> 50.0
- link wrist_pitch: mass None -> 10.0
- link wrist_roll: mass None -> 10.0
Joints:
- removed joint gripper_joint
- removed joint gripper_joint2
- joint elbow_pitch_joint: origin xyz=0 0 0.052 rpy=1.2 0 0 -> xyz=0 0 0.052 rpy=0 0 0
- joint elbow_roll_joint: origin xyz=0 0 0.089 rpy=0 0 1.2 -> xyz=0 0 0.089 rpy=0 0 0
- joint elbow_yaw_joint: origin xyz=0 0 0.072 rpy=0 -1.2 0 -> xyz=0 0 0.072 rpy=0 0 0
- joint shoulder_pitch_joint: origin xyz=0 0 0.063 rpy=1.2 0 0 -> xyz=0 0 0.063 rpy=0 0 0
- joint shoulder_roll_joint: origin xyz=0 0 0.05315 rpy=0 0 1.2 -> xyz=0 0 0.05315 rpy=0 0 0
- joint wrist_pitch_joint: origin xyz=0 0 0.0718 rpy=1.2 0 0 -> xyz=0 0 0.0718 rpy=0 0 0
- joint wrist_roll_joint: origin xyz=0 0 0.051425 rpy=0 0 1.2 -> xyz=0 0 0.051425 rpy=0 0 0
