Commit message: updated for 2017 implementation in house

File: cyton_gamma_1500_description/cyton_gamma_1500.urdf (robot description, URDF)
Before this commit: robot cyton_gamma_1500, 12 links, 11 joints
Links:
- removed link gripper_finger1
- removed link gripper_finger2
- link elbow_pitch: geometry visual mesh filename=package://cyton_gamma_1500_description/meshes/elbow_pitch.d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
- link elbow_yaw: geometry visual mesh filename=package://cyton_gamma_1500_description/meshes/elbow_yaw.dae
- link shoulder_pitch: geometry visual mesh filename=package://cyton_gamma_1500_description/meshes/shoulder_pitc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
- link shoulder_roll: geometry visual mesh filename=package://cyton_gamma_1500_description/meshes/shoulder_roll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
- link shoulder_yaw: geometry visual mesh filename=package://cyton_gamma_1500_description/meshes/shoulder_yaw.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
- link wrist_pitch: geometry visual mesh filename=package://cyton_gamma_1500_description/meshes/wrist_pitch.d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
- link wrist_roll: geometry visual mesh filename=package://cyton_gamma_1500_description/meshes/wrist_roll.dae
Joints:
- removed joint gripper_joint
- removed joint gripper_joint2
- joint wrist_pitch_joint: axis -1 0 0 -> 1 0 0

File: cyton_gamma_1500_description/cyton_gamma_1500_macros.urdf.xacro (robot description, xacro)
@@ -33,10 +33,4 @@
         </geometry>
       </collision>
-      <inertial>
-        <mass value="100.0"/>
-        <origin rpy="0 0 0" xyz="0 0 0"/>
-        <inertia ixx="1.1027" iyy="1.1027" izz="1.1027"
-                  ixy="0" ixz="0" iyz="0"/>
-      </inertial>
     </link>
     <joint name="${prefix}shoulder_roll_joint" type="revolute">
@@ -60,10 +54,4 @@
         </geometry>
       </collision>
-      <inertial>
-        <mass value="50.0"/>
-        <origin rpy="0 0 0" xyz="0 0 0"/>
-        <inertia ixx=".1027" iyy=".1027" izz=".1027"
-                  ixy="0" ixz="0" iyz="0"/>
-      </inertial>
     </link>
     <joint name="${prefix}shoulder_pitch_joint" type="revolute">
@@ -87,10 +75,4 @@
         </geometry>
       </collision>
-      <inertial>
-        <mass value="20.0"/>
-        <origin rpy="0 0 0" xyz="0 0 0"/>
-        <inertia ixx=".0827" iyy=".0827" izz=".0827"
-                  ixy="0" ixz="0" iyz="0"/>
-      </inertial>
     </link>
     <joint name="${prefix}shoulder_yaw_joint" type="revolute">
@@ -114,10 +96,4 @@
         </geometry>
       </collision>
-      <inertial>
-        <mass value="10.0"/>
-        <origin rpy="0 0 0" xyz="0 0 0"/>
-        <inertia ixx=".0627" iyy=".0627" izz=".0627"
-                  ixy="0" ixz="0" iyz="0"/>
-      </inertial>
     </link>
     <joint name="${prefix}elbow_pitch_joint" type="revolute">
@@ -141,10 +117,4 @@
         </geometry>
       </collision>
-      <inertial>
-        <mass value="10.0"/>
-        <origin rpy="0 0 0" xyz="0 0 0"/>
-        <inertia ixx=".0327" iyy=".0327" izz=".0327"
-                  ixy="0" ixz="0" iyz="0"/>
-      </inertial>
     </link>
     <joint name="${prefix}elbow_yaw_joint" type="revolute">
@@ -168,10 +138,4 @@
         </geometry>
       </collision>
-      <inertial>
-        <mass value="10.0"/>
-        <origin rpy="0 0 0" xyz="0 0 0"/>
-        <inertia ixx=".0227" iyy=".0227" izz=".0227"
-                  ixy="0" ixz="0" iyz="0"/>
-      </inertial>
     </link>
     <joint name="${prefix}wrist_pitch_joint" type="revolute">
@@ -195,10 +159,4 @@
         </geometry>
       </collision>
-      <inertial>
-        <mass value="10.0"/>
-        <origin rpy="0 0 0" xyz="0 0 0"/>
-        <inertia ixx=".0127" iyy=".0127" izz=".0127"
-                  ixy="0" ixz="0" iyz="0"/>
-      </inertial>
     </link>
     <joint name="${prefix}wrist_roll_joint" type="revolute">
@@ -222,10 +180,4 @@
         </geometry>
       </collision>
-      <inertial>
-        <mass value="10.0"/>
-        <origin rpy="0 0 0" xyz="0 0 0"/>
-        <inertia ixx=".0027" iyy=".0027" izz=".0027"
-                  ixy="0" ixz="0" iyz="0"/>
-      </inertial>
     </link>
     <joint name="${prefix}gripper_joint" type="prismatic">
@@ -249,10 +201,4 @@
         </geometry>
       </collision>
-      <inertial>
-        <mass value="1.0"/>
-        <origin rpy="0 0 0" xyz="0 0 0"/>
-        <inertia ixx=".0027" iyy=".0027" izz=".0027"
-                  ixy="0" ixz="0" iyz="0"/>
-      </inertial>
     </link>
     <joint name="${prefix}gripper_joint2" type="prismatic">
@@ -277,10 +223,4 @@
         </geometry>
       </collision>
-      <inertial>
-        <mass value="1.0"/>
-        <origin rpy="0 0 0" xyz="0 0 0"/>
-        <inertia ixx=".0027" iyy=".0027" izz=".0027"
-                  ixy="0" ixz="0" iyz="0"/>
-      </inertial>
     </link>
     <xacro:if value="${virtual_ee}"> <!-- virtual end-effector -->
@@ -303,12 +243,3 @@
     </xacro:if>
   </xacro:macro>
-  <gazebo>
-    <plugin name="gazebo_ros_control" filename="libgazebo_ros_control.so"/>
-  </gazebo>
-  <gazebo>
-    <plugin name="joint_state_publisher"
-            filename="libgazebo_ros_joint_state_publisher.so">
-      <jointName>shoulder_roll_joint, shoulder_pitch_joint, shoulder_yaw_joint, elbow_pitch_joint, elbow_yaw_joint, wrist_pitch_joint, wrist_roll_joint, gripper_joint, gripper_joint2</jointName>
-    </plugin>
-  </gazebo>
 </robot>

Commit message: fix

File: cyton_gamma_1500_description/cyton_gamma_1500.urdf (robot description, URDF)
Before this commit: robot cyton_gamma_1500, 10 links, 9 joints
Links:
- added link gripper_finger1, mass 1.0; collision box size=0.015 0.0229 0.0475; visual mesh filename=package://cyton_gamma_1500_description/meshes/gripper_finge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
- added link gripper_finger2, mass 1.0; collision box size=0.015 0.0229 0.0475; visual mesh filename=package://cyton_gamma_1500_description/meshes/gripper_finge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
- link elbow_pitch: geometry collision box size=0.0549 0.1557 0.076; visual mesh filename=package://cyton_gamma_1500_description/meshes/elbow_pitch.d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
- link elbow_yaw: geometry collision box size=0.0535 0.1160 0.0402; visual mesh filename=package://cyton_gamma_1500_description/meshes/elbow_yaw.dae
- link shoulder_pitch: geometry collision box size=0.0709 0.19363 0.083; visual mesh filename=package://cyton_gamma_1500_description/meshes/shoulder_pitc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
- link shoulder_roll: geometry collision box size=0.09829 0.18143 0.08392; visual mesh filename=package://cyton_gamma_1500_description/meshes/shoulder_roll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
- link shoulder_yaw: geometry collision box size=0.0717 0.1846 0.0756; visual mesh filename=package://cyton_gamma_1500_description/meshes/shoulder_yaw.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
- link wrist_pitch: geometry collision box size=0.026 0.0435 0.05185; visual mesh filename=package://cyton_gamma_1500_description/meshes/wrist_pitch.d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
- link wrist_roll: geometry collision box size=0.0518 0.0723 0.1004; visual mesh filename=package://cyton_gamma_1500_description/meshes/wrist_roll.dae
Joints:
- added joint gripper_joint: type prismatic, parent wrist_roll, child gripper_finger1, origin xyz=-0.01331 0.00485 0.077225 rpy=0 0 0, axis 1 0 0, limit lower=-0.008 upper=0.008 effort=100.0 velocity=1.0
- added joint gripper_joint2: type prismatic, parent wrist_roll, child gripper_finger2, origin xyz=0.0098 0.00485 0.077225 rpy=0 0 0, axis 1 0 0, limit lower=-0.008 upper=0.008 effort=100.0 velocity=1.0, mimic joint=gripper_joint multiplier=-1
- joint wrist_pitch_joint: axis 1 0 0 -> -1 0 0
